File: src/test/hardware/v0.0.1/reflow.sch (EAGLE design)
At the start: 25 parts, among them IC1 MAX31855, IC2 MAX31855, J1 1X2-3.5MM, J2 1X2-3.5MM, J3 1X2-3.5MM

Commit message: Added labels in schematic to terminal blocks.
Other:
- note added: "J1"
- note added: "J2"
- note added: "J3"
- moved on the sheet: C1, C3
Changed lines of the file:
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@@
 <text x="121.92" y="45.72" size="1.778" layer="95">GPIO2</text>
 <text x="121.92" y="30.48" size="1.778" layer="95">GPIO15</text>
+<text x="162.56" y="35.56" size="1.778" layer="95">J1</text>
+<text x="205.74" y="86.36" size="1.778" layer="95">J2</text>
+<text x="205.74" y="58.42" size="1.778" layer="95">J3</text>
 </plain>
 <instances>
@@
 <instance part="P+1" gate="1" x="45.72" y="68.58"/>
 <instance part="GND1" gate="1" x="48.26" y="0"/>
-<instance part="C1" gate="G$1" x="99.06" y="86.36"/>
-<instance part="+3V31" gate="G$1" x="99.06" y="91.44"/>
-<instance part="GND2" gate="1" x="99.06" y="78.74"/>
+<instance part="C1" gate="G$1" x="96.52" y="86.36"/>
+<instance part="+3V31" gate="G$1" x="96.52" y="91.44"/>
+<instance part="GND2" gate="1" x="96.52" y="78.74"/>
 <instance part="R3" gate="G$1" x="91.44" y="53.34"/>
 <instance part="R4" gate="G$1" x="96.52" y="43.18"/>
@@
 <instance part="JP3" gate="G$1" x="60.96" y="40.64"/>
 <instance part="C2" gate="G$1" x="106.68" y="86.36"/>
-<instance part="C3" gate="G$1" x="114.3" y="86.36"/>
+<instance part="C3" gate="G$1" x="116.84" y="86.36"/>
 <instance part="+3V32" gate="G$1" x="106.68" y="91.44"/>
-<instance part="+3V34" gate="G$1" x="114.3" y="91.44"/>
+<instance part="+3V34" gate="G$1" x="116.84" y="91.44"/>
 <instance part="GND3" gate="1" x="106.68" y="78.74"/>
-<instance part="GND4" gate="1" x="114.3" y="78.74"/>
+<instance part="GND4" gate="1" x="116.84" y="78.74"/>
 <instance part="R2" gate="G$1" x="88.9" y="60.96"/>
 <instance part="R1" gate="G$1" x="86.36" y="48.26"/>
